File: pcbs/pcb.kicad_pcb (KiCad board)
At the start: 2 copper layers, 152.3 x 118 mm, 97 parts

Commit message: update pcb and image
Routing:
- net (no net): track 5020.6 -> 5022.0 mm
Changed lines of the file:
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@@
 (segment locked (start 186.10213 203.07763) (end 188.08769 193.73632) (width 0.25) (layer B.Cu) (net 0))
 (segment locked (start 188.08769 193.73632) (end 187.93364 193.49911) (width 0.25) (layer B.Cu) (net 0))
-(segment locked (start 208.15895 192.73755) (end 206.1714 190.75) (width 0.25) (layer F.Cu) (net 0))
-(segment locked (start 206.1714 190.75) (end 202.05 190.75) (width 0.25) (layer F.Cu) (net 0))
-(via locked (at 202.05 190.75) (size 0.8) (drill 0.4) (layers "F.Cu" "B.Cu") (net 0))
-(segment locked (start 202.05 190.75) (end 194.725 183.425) (width 0.25) (layer B.Cu) (net 0))
-(segment locked (start 194.725 183.425) (end 189.15 183.425) (width 0.25) (layer B.Cu) (net 0))
-(segment locked (start 189.15 183.425) (end 188.35 182.625) (width 0.25) (layer B.Cu) (net 0))
-(segment locked (start 188.35 182.625) (end 188.35 179.1) (width 0.25) (layer B.Cu) (net 0))
-(segment locked (start 228.46846 183.76404) (end 226.45442 181.75) (width 0.25) (layer F.Cu) (net 0))
-(segment locked (start 226.45442 181.75) (end 222.825 181.75) (width 0.25) (layer F.Cu) (net 0))
-(via locked (at 222.825 181.75) (size 0.8) (drill 0.4) (layers "F.Cu" "B.Cu") (net 0))
-(segment locked (start 222.825 181.75) (end 218.125 181.75) (width 0.25) (layer B.Cu) (net 0))
-(segment locked (start 218.125 181.75) (end 206.35 169.975) (width 0.25) (layer B.Cu) (net 0))
-(segment locked (start 206.35 169.975) (end 206.35 165.1) (width 0.25) (layer B.Cu) (net 0))
-(segment locked (start 170.35 193.1) (end 171.275 194.025) (width 0.25) (layer F.Cu) (net 0))
-(segment locked (start 171.275 194.025) (end 174.85 194.025) (width 0.25) (layer F.Cu) (net 0))
-(segment locked (start 174.85 194.025) (end 176.416 192.459) (width 0.25) (layer F.Cu) (net 0))
-(segment locked (start 176.416 192.459) (end 177.559 192.459) (width 0.25) (layer F.Cu) (net 0))
-(segment locked (start 177.559 192.459) (end 180.71862 195.61862) (width 0.25) (layer F.Cu) (net 0))
-(segment locked (start 180.71862 195.61862) (end 180.71862 196.89362) (width 0.25) (layer F.Cu) (net 0))
-(segment locked (start 180.71862 196.89362) (end 186.5142 202.6892) (width 0.25) (layer F.Cu) (net 0))
-(segment locked (start 186.5142 202.6892) (end 187.64153 202.6892) (width 0.25) (layer F.Cu) (net 0))
+(segment (start 208.15895 192.73755) (end 206.1714 190.75) (width 0.25) (layer F.Cu) (net 0))
+(segment (start 206.1714 190.75) (end 202.05 190.75) (width 0.25) (layer F.Cu) (net 0))
+(via (at 202.05 190.75) (size 0.8) (drill 0.4) (layers "F.Cu" "B.Cu") (net 0))
+(segment (start 202.05 190.75) (end 194.725 183.425) (width 0.25) (layer B.Cu) (net 0))
+(segment (start 194.725 183.425) (end 189.15 183.425) (width 0.25) (layer B.Cu) (net 0))
+(segment (start 189.15 183.425) (end 188.35 182.625) (width 0.25) (layer B.Cu) (net 0))
+(segment (start 188.35 182.625) (end 188.35 179.1) (width 0.25) (layer B.Cu) (net 0))
+(segment (start 228.46846 183.76404) (end 226.45442 181.75) (width 0.25) (layer F.Cu) (net 0))
+(segment (start 226.45442 181.75) (end 222.825 181.75) (width 0.25) (layer F.Cu) (net 0))
+(via (at 222.825 181.75) (size 0.8) (drill 0.4) (layers "F.Cu" "B.Cu") (net 0))
+(segment (start 222.825 181.75) (end 218.125 181.75) (width 0.25) (layer B.Cu) (net 0))
+(segment (start 218.125 181.75) (end 206.35 169.975) (width 0.25) (layer B.Cu) (net 0))
+(segment (start 206.35 169.975) (end 206.35 165.1) (width 0.25) (layer B.Cu) (net 0))
+(segment (start 170.35 193.1) (end 171.275 194.025) (width 0.25) (layer F.Cu) (net 0))
+(segment (start 171.275 194.025) (end 174.85 194.025) (width 0.25) (layer F.Cu) (net 0))
+(segment (start 174.85 194.025) (end 176.416 192.459) (width 0.25) (layer F.Cu) (net 0))
+(segment (start 176.416 192.459) (end 177.559 192.459) (width 0.25) (layer F.Cu) (net 0))
+(segment (start 177.559 192.459) (end 179.675 194.575) (width 0.25) (layer F.Cu) (net 0))
+(segment (start 179.675 194.575) (end 179.675 195.85) (width 0.25) (layer F.Cu) (net 0))
+(segment (start 179.675 195.85) (end 186.5142 202.6892) (width 0.25) (layer F.Cu) (net 0))
+(segment (start 186.5142 202.6892) (end 187.64153 202.6892) (width 0.25) (layer F.Cu) (net 0))
+(segment (start 187.64153 202.6892) (end 188.4187 203.88594) (width 0.25) (layer F.Cu) (net 0))
 (segment locked (start 187.93364 193.49911) (end 186.925 192.49047) (width 0.25) (layer B.Cu) (net 0))
 (segment locked (start 186.925 192.49047) (end 186.925 167.5) (width 0.25) (layer B.Cu) (net 0))
